File: Hardware-Main/Squirco Logic v1.0.sch (EAGLE design)
At the start: 77 parts, among them IC1 LP2985-33DBVR, U3 ATMEGA256RFR2, Y1 16MHz, Y3 32.768kHz, Y4 32MHz

Commit message: Merge remote-tracking branch 'origin/master'
Conflicts:
	Hardware-Extras/README.md
Parts:
- C4: value (none) -> DNI
- renumbered U$1 to ANT2, U$2 to U4, U$3 to B2
Other:
- moved on the sheet: C4
